File: hdw/PIC32MZ_TFT_Demo/PGOOD_LEDs.sch (KiCad schematic (older format))
At the start: 8 parts, among them U1803 74LVC1G06, U1806 74LVC1G06

Commit message: Started PCB layout
Parts:
- renumbered C1803 to C901, C1806 to C902, D1802 to D901, D1805 to D902, R1802 to R901, R1805 to R902, U1803 to U901, U1806 to U902
Changed lines of the file:
@@
 EESchema Schematic File Version 4
+LIBS:PIC32MZ_TFT_Demo-cache
 EELAYER 30 0
 EELAYER END
 $Descr A 11000 8500
 encoding utf-8
-Sheet 9 11
-Title "Pulse Oximeter"
-Date "2019-01-03"
+Sheet 9 13
+Title ""
+Date "2020-07-04"
 Rev "A"
 Comp "Drew Maatman"
@@
 AR Path="/5CB7A8BC/5CB97030" Ref="C?"  Part="1"
 AR Path="/5CB7A8C3/5CB97030" Ref="C?"  Part="1"
-AR Path="/5EAE4ADE/5CB97030" Ref="C1806"  Part="1"
-AR Path="/5EE6161A/5CB97030" Ref="C1806"  Part="1"
-F 0 "C1806" H 8895 2280 50  0000 L CNN
+AR Path="/5EAE4ADE/5CB97030" Ref="C?"  Part="1"
+AR Path="/5EE6161A/5CB97030" Ref="C902"  Part="1"
+F 0 "C902" H 8895 2280 50  0000 L CNN
 F 1 "0.1uF" H 8895 2080 50  0000 L CNN
 F 2 "Capacitors_SMD:C_0402" H 8908 2030 50  0001 C CNN
@@
 AR Path="/5CB7A8BC/5CB9703B" Ref="D?"  Part="1"
 AR Path="/5CB7A8C3/5CB9703B" Ref="D?"  Part="1"
-AR Path="/5EAE4ADE/5CB9703B" Ref="D1805"  Part="1"
-AR Path="/5EE6161A/5CB9703B" Ref="D1805"  Part="1"
-F 0 "D1805" V 9589 2483 50  0000 R CNN
+AR Path="/5EAE4ADE/5CB9703B" Ref="D?"  Part="1"
+AR Path="/5EE6161A/5CB9703B" Ref="D902"  Part="1"
+F 0 "D902" V 9589 2483 50  0000 R CNN
 F 1 "Green" V 9498 2483 50  0000 R CNN
 F 2 "LEDs:LED_0402" H 9550 2600 50  0001 C CNN
@@
 AR Path="/5CB7A8BC/5CB9704B" Ref="R?"  Part="1"
 AR Path="/5CB7A8C3/5CB9704B" Ref="R?"  Part="1"
-AR Path="/5EAE4ADE/5CB9704B" Ref="R1805"  Part="1"
-AR Path="/5EE6161A/5CB9704B" Ref="R1805"  Part="1"
-F 0 "R1805" H 9490 2300 50  0000 R CNN
+AR Path="/5EAE4ADE/5CB9704B" Ref="R?"  Part="1"
+AR Path="/5EE6161A/5CB9704B" Ref="R902"  Part="1"
+F 0 "R902" H 9490 2300 50  0000 R CNN
 F 1 "1k" V 9550 2300 50  0000 C CNN
 F 2 "Resistors_SMD:R_0402" H 9550 2300 50  0001 C CNN
@@
 AR Path="/5CB7A8BC/5CB97055" Ref="#PWR?"  Part="1"
 AR Path="/5CB7A8C3/5CB97055" Ref="#PWR?"  Part="1"
-AR Path="/5EAE4ADE/5CB97055" Ref="#PWR01825"  Part="1"
-AR Path="/5EE6161A/5CB97055" Ref="#PWR01825"  Part="1"
-F 0 "#PWR01825" H 9550 2000 50  0001 C CNN
+AR Path="/5EAE4ADE/5CB97055" Ref="#PWR?"  Part="1"
+AR Path="/5EE6161A/5CB97055" Ref="#PWR0910"  Part="1"
+F 0 "#PWR0910" H 9550 2000 50  0001 C CNN
 F 1 "+3.3V" H 9550 2290 50  0000 C CNN
 F 2 "" H 9550 2150 50  0001 C CNN
@@
 AR Path="/5CB7A8BC/5CB9705F" Ref="#PWR?"  Part="1"
 AR Path="/5CB7A8C3/5CB9705F" Ref="#PWR?"  Part="1"
-AR Path="/5EAE4ADE/5CB9705F" Ref="#PWR01823"  Part="1"
-AR Path="/5EE6161A/5CB9705F" Ref="#PWR01823"  Part="1"
-F 0 "#PWR01823" H 8980 2620 50  0001 C CNN
+AR Path="/5EAE4ADE/5CB9705F" Ref="#PWR?"  Part="1"
+AR Path="/5EE6161A/5CB9705F" Ref="#PWR0908"  Part="1"
+F 0 "#PWR0908" H 8980 2620 50  0001 C CNN
 F 1 "+3.3V" H 8980 2910 50  0000 C CNN
 F 2 "" H 8980 2770 50  0001 C CNN
@@
 AR Path="/5CB7A8BC/5CB97069" Ref="#PWR?"  Part="1"
 AR Path="/5CB7A8C3/5CB97069" Ref="#PWR?"  Part="1"
-AR Path="/5EAE4ADE/5CB97069" Ref="#PWR01821"  Part="1"
-AR Path="/5EE6161A/5CB97069" Ref="#PWR01821"  Part="1"
-F 0 "#PWR01821" H 8870 1880 50  0001 C CNN
+AR Path="/5EAE4ADE/5CB97069" Ref="#PWR?"  Part="1"
+AR Path="/5EE6161A/5CB97069" Ref="#PWR0906"  Part="1"
+F 0 "#PWR0906" H 8870 1880 50  0001 C CNN
 F 1 "+3.3V" H 8870 2170 50  0000 C CNN
 F 2 "" H 8870 2030 50  0001 C CNN
@@
 AR Path="/5CB7A8BC/5CB97073" Ref="#PWR?"  Part="1"
 AR Path="/5CB7A8C3/5CB97073" Ref="#PWR?"  Part="1"
-AR Path="/5EAE4ADE/5CB97073" Ref="#PWR01824"  Part="1"
-AR Path="/5EE6161A/5CB97073" Ref="#PWR01824"  Part="1"
-F 0 "#PWR01824" H 8980 2720 50  0001 C CNN
+AR Path="/5EAE4ADE/5CB97073" Ref="#PWR?"  Part="1"
+AR Path="/5EE6161A/5CB97073" Ref="#PWR0909"  Part="1"
+F 0 "#PWR0909" H 8980 2720 50  0001 C CNN
 F 1 "GND" H 8980 2820 50  0000 C CNN
 F 2 "" H 8980 2970 50  0001 C CNN
@@
 AR Path="/5CB7A8BC/5CB9707D" Ref="#PWR?"  Part="1"
 AR Path="/5CB7A8C3/5CB9707D" Ref="#PWR?"  Part="1"
-AR Path="/5EAE4ADE/5CB9707D" Ref="#PWR01822"  Part="1"
-AR Path="/5EE6161A/5CB9707D" Ref="#PWR01822"  Part="1"
-F 0 "#PWR01822" H 8870 2080 50  0001 C CNN
+AR Path="/5EAE4ADE/5CB9707D" Ref="#PWR?"  Part="1"
+AR Path="/5EE6161A/5CB9707D" Ref="#PWR0907"  Part="1"
+F 0 "#PWR0907" H 8870 2080 50  0001 C CNN
 F 1 "GND" H 8870 2180 50  0000 C CNN
 F 2 "" H 8870 2330 50  0001 C CNN
@@
 AR Path="/5CB7A8BC/5E1829A4" Ref="C?"  Part="1"
 AR Path="/5CB7A8C3/5E1829A4" Ref="C?"  Part="1"
-AR Path="/5EAE4ADE/5E1829A4" Ref="C1803"  Part="1"
-AR Path="/5EE6161A/5E1829A4" Ref="C1803"  Part="1"
-F 0 "C1803" H 2895 3780 50  0000 L CNN
+AR Path="/5EAE4ADE/5E1829A4" Ref="C?"  Part="1"
+AR Path="/5EE6161A/5E1829A4" Ref="C901"  Part="1"
+F 0 "C901" H 2895 3780 50  0000 L CNN
 F 1 "0.1uF" H 2895 3580 50  0000 L CNN
 F 2 "Capacitors_SMD:C_0402" H 2908 3530 50  0001 C CNN
@@
 AR Path="/5CB7A8BC/5E1829AF" Ref="D?"  Part="1"
 AR Path="/5CB7A8C3/5E1829AF" Ref="D?"  Part="1"
-AR Path="/5EAE4ADE/5E1829AF" Ref="D1802"  Part="1"
-AR Path="/5EE6161A/5E1829AF" Ref="D1802"  Part="1"
-F 0 "D1802" V 3589 3983 50  0000 R CNN
+AR Path="/5EAE4ADE/5E1829AF" Ref="D?"  Part="1"
+AR Path="/5EE6161A/5E1829AF" Ref="D901"  Part="1"
+F 0 "D901" V 3589 3983 50  0000 R CNN
 F 1 "Green" V 3498 3983 50  0000 R CNN
 F 2 "LEDs:LED_0402" H 3550 4100 50  0001 C CNN
@@
 AR Path="/5CB7A8BC/5E1829BF" Ref="R?"  Part="1"
 AR Path="/5CB7A8C3/5E1829BF" Ref="R?"  Part="1"
-AR Path="/5EAE4ADE/5E1829BF" Ref="R1802"  Part="1"
-AR Path="/5EE6161A/5E1829BF" Ref="R1802"  Part="1"
-F 0 "R1802" H 3490 3800 50  0000 R CNN
+AR Path="/5EAE4ADE/5E1829BF" Ref="R?"  Part="1"
+AR Path="/5EE6161A/5E1829BF" Ref="R901"  Part="1"
+F 0 "R901" H 3490 3800 50  0000 R CNN
 F 1 "1k" V 3550 3800 50  0000 C CNN
 F 2 "Resistors_SMD:R_0402" H 3550 3800 50  0001 C CNN
@@
 AR Path="/5CB7A8BC/5E1829C9" Ref="#PWR?"  Part="1"
 AR Path="/5CB7A8C3/5E1829C9" Ref="#PWR?"  Part="1"
-AR Path="/5EAE4ADE/5E1829C9" Ref="#PWR01810"  Part="1"
-AR Path="/5EE6161A/5E1829C9" Ref="#PWR01810"  Part="1"
-F 0 "#PWR01810" H 3550 3500 50  0001 C CNN
+AR Path="/5EAE4ADE/5E1829C9" Ref="#PWR?"  Part="1"
+AR Path="/5EE6161A/5E1829C9" Ref="#PWR0905"  Part="1"
+F 0 "#PWR0905" H 3550 3500 50  0001 C CNN
 F 1 "+3.3V" H 3550 3790 50  0000 C CNN
 F 2 "" H 3550 3650 50  0001 C CNN
@@
 AR Path="/5CB7A8BC/5E1829D3" Ref="#PWR?"  Part="1"
 AR Path="/5CB7A8C3/5E1829D3" Ref="#PWR?"  Part="1"
-AR Path="/5EAE4ADE/5E1829D3" Ref="#PWR01808"  Part="1"
-AR Path="/5EE6161A/5E1829D3" Ref="#PWR01808"  Part="1"
-F 0 "#PWR01808" H 2980 4120 50  0001 C CNN
+AR Path="/5EAE4ADE/5E1829D3" Ref="#PWR?"  Part="1"
+AR Path="/5EE6161A/5E1829D3" Ref="#PWR0903"  Part="1"
+F 0 "#PWR0903" H 2980 4120 50  0001 C CNN
 F 1 "+3.3V" H 2980 4410 50  0000 C CNN
 F 2 "" H 2980 4270 50  0001 C CNN
@@
 AR Path="/5CB7A8BC/5E1829DD" Ref="#PWR?"  Part="1"
 AR Path="/5CB7A8C3/5E1829DD" Ref="#PWR?"  Part="1"
-AR Path="/5EAE4ADE/5E1829DD" Ref="#PWR01805"  Part="1"
-AR Path="/5EE6161A/5E1829DD" Ref="#PWR01805"  Part="1"
-F 0 "#PWR01805" H 2870 3380 50  0001 C CNN
+AR Path="/5EAE4ADE/5E1829DD" Ref="#PWR?"  Part="1"
+AR Path="/5EE6161A/5E1829DD" Ref="#PWR0901"  Part="1"
+F 0 "#PWR0901" H 2870 3380 50  0001 C CNN
 F 1 "+3.3V" H 2870 3670 50  0000 C CNN
 F 2 "" H 2870 3530 50  0001 C CNN
@@
 AR Path="/5CB7A8BC/5E1829E7" Ref="#PWR?"  Part="1"
 AR Path="/5CB7A8C3/5E1829E7" Ref="#PWR?"  Part="1"
-AR Path="/5EAE4ADE/5E1829E7" Ref="#PWR01809"  Part="1"
-AR Path="/5EE6161A/5E1829E7" Ref="#PWR01809"  Part="1"
-F 0 "#PWR01809" H 2980 4220 50  0001 C CNN
+AR Path="/5EAE4ADE/5E1829E7" Ref="#PWR?"  Part="1"
+AR Path="/5EE6161A/5E1829E7" Ref="#PWR0904"  Part="1"
+F 0 "#PWR0904" H 2980 4220 50  0001 C CNN
 F 1 "GND" H 2980 4320 50  0000 C CNN
 F 2 "" H 2980 4470 50  0001 C CNN
@@
 AR Path="/5CB7A8BC/5E1829F1" Ref="#PWR?"  Part="1"
 AR Path="/5CB7A8C3/5E1829F1" Ref="#PWR?"  Part="1"
-AR Path="/5EAE4ADE/5E1829F1" Ref="#PWR01806"  Part="1"
-AR Path="/5EE6161A/5E1829F1" Ref="#PWR01806"  Part="1"
-F 0 "#PWR01806" H 2870 3580 50  0001 C CNN
+AR Path="/5EAE4ADE/5E1829F1" Ref="#PWR?"  Part="1"
+AR Path="/5EE6161A/5E1829F1" Ref="#PWR0902"  Part="1"
+F 0 "#PWR0902" H 2870 3580 50  0001 C CNN
 F 1 "GND" H 2870 3680 50  0000 C CNN
 F 2 "" H 2870 3830 50  0001 C CNN
@@
 POS5_USB_PGOOD
 $Comp
-L Custom_Library:74LVC1G06_Power U1806
+L Custom_Library:74LVC1G06_Power U902
 U 1 1 5EBAE6FA
 P 8980 2870
-F 0 "U1806" H 9080 3020 50  0000 L CNN
+F 0 "U902" H 9080 3020 50  0000 L CNN
 F 1 "74LVC1G06" H 9080 2770 50  0000 L CNN
 F 2 "TO_SOT_Packages_SMD:SOT-353_SC-70-5" H 8980 2920 50  0001 C CNN
@@
 $EndComp
 $Comp
-L Custom_Library:74LVC1G06_Power U1803
+L Custom_Library:74LVC1G06_Power U901
 U 1 1 5EBAEFAB
 P 2980 4370
-F 0 "U1803" H 3080 4520 50  0000 L CNN
+F 0 "U901" H 3080 4520 50  0000 L CNN
 F 1 "74LVC1G06" H 3080 4270 50  0000 L CNN
 F 2 "TO_SOT_Packages_SMD:SOT-353_SC-70-5" H 2980 4420 50  0001 C CNN
