File: hdw/PIC32MZ_TFT_Demo/PIC32MZ_Bypass.sch (KiCad schematic (older format))
At the start: 31 parts

Commit message: Started PCB layout
Parts:
- removed C501: 22uF, Capacitors_SMD:C_1206, symbol Custom_Library:C_Custom
- added C601: 100uF, Capacitors_SMD:C_1206, symbol Custom_Library:C_Custom
- renumbered C502 to C602, C503 to C603, C504 to C604, C505 to C605, C506 to C606, C507 to C607, C508 to C608, C509 to C609, C510 to C610, C511 to C611, C512 to C612, C513 to C613, C514 to C614, C515 to C615, C516 to C616, C517 to C617, C518 to C618, C519 to C619, C520 to C620, C521 to C621, C522 to C622, C523 to C623, C524 to C624, C525 to C625, C526 to C626, C527 to C627, C528 to C628, C529 to C629, L501 to L601, L502 to L602
Connections:
- net +3V3: now also C601.1
- net GND: now also C601.2
- net +3.3VA renamed +3.3VA_MZ
- net GNDA renamed GNDA_MZ
