File: hdw/PIC32MZ_TFT_Demo/PIC32MZ_Clocking.sch (KiCad schematic (older format))
At the start: 17 parts, among them X701 ASE-8.000MHz, X702 ECS-327KE

Commit message: Started PCB layout
Parts:
- removed C702: 0.1uF, Capacitors_SMD:C_0402, symbol Custom_Library:C_Custom
- removed C704: 10nF, Capacitors_SMD:C_0402, symbol Custom_Library:C_Custom
- removed C706: 1nF, Capacitors_SMD:C_0402, symbol Custom_Library:C_Custom
- removed L702: 600R 0.5A, Inductors_SMD:L_0402, symbol Device:Ferrite_Bead
- removed R703: 100, Resistors_SMD:R_0402, symbol Custom_Library:R_Custom
- removed R705: 10k, Resistors_SMD:R_0402, symbol Custom_Library:R_Custom
- removed X702: ECS-327KE, Custom Footprints Library:ECS-327KE, symbol Custom_Library:ECS-327KE
- gave numbers to parts that had none: 2
- renumbered C701 to C501, C703 to C502, C705 to C503, L701 to L501, R701 to R502, R702 to R503, R704 to R504, X701 to X501
