File: hdw/PIC32MZ_TFT_Demo/PIC32MZ_TFT_Demo.sch (KiCad schematic (older format))
At the start: 0 parts

Commit message: Started PCB layout
Other:
- note removed: "Add Mechanical Sheet"
Changed lines of the file:
@@
 EESchema Schematic File Version 4
+LIBS:PIC32MZ_TFT_Demo-cache
 EELAYER 30 0
 EELAYER END
 $Descr A 11000 8500
 encoding utf-8
-Sheet 1 11
+Sheet 1 13
 Title ""
-Date ""
-Rev ""
-Comp ""
+Date "2020-07-04"
+Rev "A"
+Comp "Drew Maatman"
 Comment1 ""
 Comment2 ""
@@
 F1 "USB_UART_Bridge.sch" 50
 $EndSheet
-Text Notes 7710 4910 0    250  ~ 50
-Add Mechanical Sheet
 $Sheet
 S 2030 3910 500  150
@@
 F1 "TFT_Screen.sch" 50
 $EndSheet
+$Sheet
+S 2030 4960 500  150
+U 5EF9E990
+F0 "SPI Flash" 50
+F1 "SPI_Flash.sch" 50
+$EndSheet
+$Sheet
+S 2030 5310 500  150
+U 5F00C3A2
+F0 "Mechanical" 50
+F1 "Mechanical.sch" 50
+$EndSheet
 $EndSCHEMATC
