File: hdw/PIC32MZ_TFT_Demo/Status_LEDs.sch (KiCad schematic (older format))
At the start: 20 parts, among them U1901 74LVC1G06, U1902 74LVC1G06, U1903 74LVC1G06, U1904 74LVC1G06

Commit message: Started PCB layout
Parts:
- renumbered C1901 to C1001, C1902 to C1002, C1903 to C1003, C1904 to C1004, D1901 to D1001, D1902 to D1002, D1903 to D1003, D1904 to D1004, R1901 to R1001, R1902 to R1002, R1903 to R1003, R1904 to R1004, R1905 to R1005, R1906 to R1006, R1907 to R1007, R1908 to R1008, U1901 to U1001, U1902 to U1002, U1903 to U1003, U1904 to U1004
