File: hdw/PIC32MZ_TFT_Demo/USB_UART_Bridge.sch (KiCad schematic (older format))
At the start: 25 parts, among them J1201 USB_B_Mini, U1201 TLV6700, U1202 FT234XD, U1203 TPD3S014DBVR

Commit message: Started PCB layout
Parts:
- renumbered C1201 to C801, C1202 to C802, C1203 to C803, C1204 to C804, C1205 to C805, C1206 to C806, C1207 to C807, C1208 to C808, C1209 to C809, D1201 to D801, DOC1201 to DOC801, J1201 to J801, L1201 to L801, L1202 to L802, R1201 to R801, R1202 to R802, R1203 to R803, R1204 to R804, R1207 to R805, R1208 to R806, R1210 to R807, TP1201 to TP801, U1201 to U801, U1202 to U802, U1203 to U803
