File: hdw/PIC32MZ_TFT_Demo/PIC32MZ_TFT_Demo.kicad_pcb (KiCad board)
At the start: 2 copper layers, 170 parts, among them J1101 TFT FFC, J201 +12V IN, J401 PICKIT4, J801 USB_B_Mini, Q401 BSS214NW, SW401 MRST, U1001 74LVC1G06, U1002 74LVC1G06, U1003 74LVC1G06, U1004 74LVC1G06, U1101 SiP32431DR3, U1201 74LVC1G07, U1202 SST25VF080B-50-4I-S2AF, U301 TPS62150, U401 74LVC1G06, U701 PIC32MZ2048EFG100_IPT, U801 TLV6700, U802 FT234XD, U803 TPD3S014DBVR, U901 74LVC1G06, U902 74LVC1G06, X501 ASE-8.000MHz

Commit message: More board part arrangement
Parts:
- C1102, C1104, C1105, C1106, R1101, R1102, R1108, R1109, R1110, R1111, R1206, R1207, R1208, R1209, R1211, R502, R504, RN1103, RN1104: moved to B.Cu
- moved R901 269.9 mm to (139.7, 21.7)
- moved C902 269.7 mm to (136.7, 29.3), turned to 180 degrees
- moved R902 269.0 mm to (139.8, 26.8)
- moved D901 267.3 mm to (139.7, 23.1)
- moved C901 267.0 mm to (136.7, 24.3), turned to 180 degrees
- moved U902 266.9 mm to (136.7, 27.4)
- moved U901 264.3 mm to (136.7, 22.4)
- moved D902 259.9 mm to (139.8, 28.1)
- moved R1212 154.4 mm to (212.1, 43.5), turned to 180 degrees
- moved R1211 153.9 mm to (212.1, 43.5), turned to 180 degrees
- moved R1208 153.7 mm to (212.1, 42.2)
- moved R1201 152.9 mm to (214.9, 37.5)
- moved R1209 151.8 mm to (212.1, 44.8)
- moved C1201 151.0 mm to (212.0, 40.1), turned to 180 degrees
- moved R1204 150.6 mm to (212.1, 42.2), turned to 180 degrees
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Connections:
- RN1101 pad 1: TFT_DB0 -> TFT_DB7
- RN1101 pad 10: Net-(J1101-Pad20) -> Net-(J1101-Pad15)
- RN1101 pad 11: Net-(J1101-Pad19) -> Net-(J1101-Pad16)
- RN1101 pad 12: Net-(J1101-Pad18) -> Net-(J1101-Pad17)
- RN1101 pad 13: Net-(J1101-Pad17) -> Net-(J1101-Pad18)
- RN1101 pad 14: Net-(J1101-Pad16) -> Net-(J1101-Pad19)
- RN1101 pad 15: Net-(J1101-Pad15) -> Net-(J1101-Pad20)
- RN1101 pad 16: Net-(J1101-Pad14) -> Net-(J1101-Pad21)
- RN1101 pad 2: TFT_DB1 -> TFT_DB6
- RN1101 pad 3: TFT_DB2 -> TFT_DB5
- RN1101 pad 4: TFT_DB3 -> TFT_DB4
- RN1101 pad 5: TFT_DB4 -> TFT_DB3
- RN1101 pad 6: TFT_DB5 -> TFT_DB2
- RN1101 pad 7: TFT_DB6 -> TFT_DB1
- RN1101 pad 8: TFT_DB7 -> TFT_DB0
- RN1101 pad 9: Net-(J1101-Pad21) -> Net-(J1101-Pad14)
- RN1102 pad 1: TFT_DB8 -> TFT_DB15
- RN1102 pad 10: Net-(J1101-Pad28) -> Net-(J1101-Pad23)
- RN1102 pad 11: Net-(J1101-Pad27) -> Net-(J1101-Pad24)
- RN1102 pad 12: Net-(J1101-Pad26) -> Net-(J1101-Pad25)
- RN1102 pad 13: Net-(J1101-Pad25) -> Net-(J1101-Pad26)
- RN1102 pad 14: Net-(J1101-Pad24) -> Net-(J1101-Pad27)
- RN1102 pad 15: Net-(J1101-Pad23) -> Net-(J1101-Pad28)
- RN1102 pad 16: Net-(J1101-Pad22) -> Net-(J1101-Pad29)
- RN1102 pad 2: TFT_DB9 -> TFT_DB14
- RN1102 pad 3: TFT_DB10 -> TFT_DB13
- RN1102 pad 4: TFT_DB11 -> TFT_DB12
- RN1102 pad 5: TFT_DB12 -> TFT_DB11
- RN1102 pad 6: TFT_DB13 -> TFT_DB10
- RN1102 pad 7: TFT_DB14 -> TFT_DB9
- RN1102 pad 8: TFT_DB15 -> TFT_DB8
- RN1102 pad 9: Net-(J1101-Pad29) -> Net-(J1101-Pad22)
- RN1103 pad 10: Net-(J1101-Pad28) -> Net-(J1101-Pad23)
- RN1103 pad 11: Net-(J1101-Pad27) -> Net-(J1101-Pad24)
- RN1103 pad 12: Net-(J1101-Pad26) -> Net-(J1101-Pad25)
- RN1103 pad 13: Net-(J1101-Pad25) -> Net-(J1101-Pad26)
- RN1103 pad 14: Net-(J1101-Pad24) -> Net-(J1101-Pad27)
- RN1103 pad 15: Net-(J1101-Pad23) -> Net-(J1101-Pad28)
- RN1103 pad 16: Net-(J1101-Pad22) -> Net-(J1101-Pad29)
- RN1103 pad 9: Net-(J1101-Pad29) -> Net-(J1101-Pad22)
- RN1104 pad 10: Net-(J1101-Pad20) -> Net-(J1101-Pad15)
- RN1104 pad 11: Net-(J1101-Pad19) -> Net-(J1101-Pad16)
- RN1104 pad 12: Net-(J1101-Pad18) -> Net-(J1101-Pad17)
- RN1104 pad 13: Net-(J1101-Pad17) -> Net-(J1101-Pad18)
- RN1104 pad 14: Net-(J1101-Pad16) -> Net-(J1101-Pad19)
- RN1104 pad 15: Net-(J1101-Pad15) -> Net-(J1101-Pad20)
- RN1104 pad 16: Net-(J1101-Pad14) -> Net-(J1101-Pad21)
- RN1104 pad 9: Net-(J1101-Pad21) -> Net-(J1101-Pad14)
Other:
- board text added: "+3.3V"
- board text added: "+5V USB"
- board text added: "Flash CE"
- board text added: "PGOOD:"
- board text added: "REFCLK1"
